File: AYOMSM - VCA Control Board.sch (KiCad schematic (older format))
At the start: 10 parts, among them J1 SIGNAL_OUT, J2 CV1, J3 CV2, J4 SIGNAL_IN, J5 CONN_1, J6 CONN_2, SW1 SW_SPDT

Commit message: Added test point for offset potentiometer
Parts:
- added TP1: OFFSET_ADJ_TP, TestPoint:TestPoint_2Pads_Pitch5.08mm_Drill1.3mm, symbol Connector:TestPoint_2Pole
Connections:
- net GND: now also TP1.1
- net OFFSET_ADJ: now also TP1.2
Changed lines of the file:
@@
 	-1   0    0    1
 $EndComp
+$Comp
+L Connector:TestPoint_2Pole TP1
+U 1 1 5EC92ABA
+P 3825 3200
+F 0 "TP1" H 3825 3395 50  0000 C CNN
+F 1 "OFFSET_ADJ_TP" H 3825 3304 50  0000 C CNN
+F 2 "TestPoint:TestPoint_2Pads_Pitch5.08mm_Drill1.3mm" H 3825 3200 50  0001 C CNN
+F 3 "~" H 3825 3200 50  0001 C CNN
+	1    3825 3200
+	1    0    0    -1
+$EndComp
+Text Label 4025 3200 0    50   ~ 0
+OFFSET_ADJ
+$Comp
+L power:GND #PWR0112
+U 1 1 5EC935CF
+P 3625 3200
+F 0 "#PWR0112" H 3625 2950 50  0001 C CNN
+F 1 "GND" H 3630 3027 50  0000 C CNN
+F 2 "" H 3625 3200 50  0001 C CNN
+F 3 "" H 3625 3200 50  0001 C CNN
+	1    3625 3200
+	0    1    1    0
+$EndComp
 $EndSCHEMATC

Commit message: Updated layout and added SPDT switch model
Parts:
- SW1: footprint Connector_PinHeader_2.54mm:PinHeader_1x03_P2.54mm_Vertical -> Custom:Mini_Toggle_Switch_SPDT_ON-ON
Changed lines of the file:
@@
 F 0 "SW1" H 5450 4085 50  0000 C CNN
 F 1 "SW_SPDT" H 5450 3994 50  0000 C CNN
-F 2 "Connector_PinHeader_2.54mm:PinHeader_1x03_P2.54mm_Vertical" H 5450 3800 50  0001 C CNN
+F 2 "Custom:Mini_Toggle_Switch_SPDT_ON-ON" H 5450 3800 50  0001 C CNN
 F 3 "~" H 5450 3800 50  0001 C CNN
 	1    5450 3800
