File: KiCad/AYOMSM - VCA Control Board.sch (KiCad schematic (older format))
At the start: 11 parts, among them J1 SIGNAL_OUT, J2 CV1, J3 CV2, J4 SIGNAL_IN, J5 CONN_1, J6 CONN_2, SW1 SW_SPDT

Commit message: Restructured repo, added Gerbers, Gerber archive, and SVG exports
Connections:
- net TRIM_1: now also RV2.2
- net TRIM_2: no longer RV2.2
Changed lines of the file:
@@
 TRIM_1
 Wire Wire Line
-	3800 3675 3800 3575
+	3800 3675 3800 3625
 Wire Wire Line
-	3950 3825 4050 3825
+	3950 3825 4000 3825
 Wire Wire Line
 	3800 3975 3800 4100
-Text Label 4050 3825 0    50   ~ 0
-TRIM_2
 Text Label 3800 4100 0    50   ~ 0
 TRIM_3
@@
 	0    1    1    0
 $EndComp
+Wire Wire Line
+	3800 3625 4000 3625
+Wire Wire Line
+	4000 3625 4000 3825
+Connection ~ 3800 3625
+Wire Wire Line
+	3800 3625 3800 3575
 $EndSCHEMATC

Commit message: Updated Gerbers and archive
Connections:
- net TRIM_2: no longer names the net of J6.5 (Pin_5)
- no-connect marks 0 -> 1
Changed lines of the file:
@@
 Text Label 8900 2675 2    50   ~ 0
 TRIM_1
-Text Label 8900 2775 2    50   ~ 0
-TRIM_2
 Text Label 8900 2875 2    50   ~ 0
 TRIM_3
@@
 Wire Wire Line
 	3800 3625 3800 3575
+NoConn ~ 8900 2775
 $EndSCHEMATC

Commit message: Updated Gerbers
Connections:
- net GND: no longer J1.2, J2.2, J3.2, J4.2
- no-connect marks 1 -> 5
Changed lines of the file:
@@
-$EndComp
-$Comp
-L Thonkiconn:fuzzySI_thonkiconn J4
-U 1 1 5EC4DB7C
-P 2375 3350
-F 0 "J4" H 2353 3675 50  0000 C CNN
-F 1 "SIGNAL_IN" H 2353 3584 50  0000 C CNN
-F 2 "Thonkiconn:thonkiconn_fuzzySi" H 2625 3450 50  0001 C CNN
-F 3 "" H 2625 3450 50  0001 C CNN
-	1    2375 3350
-	1    0    0    -1
 $EndComp
 $Comp
@@
 	1    0    0    -1
 $EndComp
-Wire Wire Line
-	2175 1875 2175 1925
-Wire Wire Line
-	2575 1775 2625 1775
-Wire Wire Line
-	2625 1775 2625 1925
-Wire Wire Line
-	2625 1925 2175 1925
-Connection ~ 2175 1925
-Wire Wire Line
-	2175 1925 2175 2000
 $Comp
 L power:GND #PWR0107
@@
 	1    0    0    -1
 $EndComp
-Wire Wire Line
-	2175 2675 2175 2725
-Wire Wire Line
-	2575 2575 2625 2575
-Wire Wire Line
-	2625 2575 2625 2725
-Wire Wire Line
-	2625 2725 2175 2725
-Connection ~ 2175 2725
-Wire Wire Line
-	2175 2725 2175 2775
 Text Label 2575 1675 0    50   ~ 0
 CV1
@@
 	1    0    0    -1
 $EndComp
-Wire Wire Line
-	2175 3575 2175 3500
-Wire Wire Line
-	2575 3350 2625 3350
-Wire Wire Line
-	2625 3350 2625 3500
-Wire Wire Line
-	2625 3500 2175 3500
-Connection ~ 2175 3500
-Wire Wire Line
-	2175 3500 2175 3450
 Text Label 2575 3250 0    50   ~ 0
 SIGNAL_IN
@@
 	1    0    0    -1
 $EndComp
-Wire Wire Line
-	2550 4425 2550 4350
-Wire Wire Line
-	2150 4200 2075 4200
-Wire Wire Line
-	2075 4200 2075 4350
-Wire Wire Line
-	2075 4350 2550 4350
-Connection ~ 2550 4350
-Wire Wire Line
-	2550 4350 2550 4300
 Text Label 2150 4100 2    50   ~ 0
 SIGNAL_OUT
@@
 	3800 3625 3800 3575
 NoConn ~ 8900 2775
+Wire Wire Line
+	2175 1875 2175 2000
+Wire Wire Line
+	2175 2675 2175 2775
+$Comp
+L Thonkiconn:fuzzySI_thonkiconn J4
+U 1 1 5EC4DB7C
+P 2375 3350
+F 0 "J4" H 2353 3675 50  0000 C CNN
+F 1 "SIGNAL_IN" H 2353 3584 50  0000 C CNN
+F 2 "Thonkiconn:thonkiconn_fuzzySi" H 2625 3450 50  0001 C CNN
+F 3 "" H 2625 3450 50  0001 C CNN
+	1    2375 3350
+	1    0    0    -1
+$EndComp
+Wire Wire Line
+	2175 3450 2175 3575
+Wire Wire Line
+	2550 4300 2550 4425
+NoConn ~ 2575 1775
+NoConn ~ 2575 2575
+NoConn ~ 2575 3350
+NoConn ~ 2150 4200
 $EndSCHEMATC
